Commit message: dev

File: robots/omp/rmpflow_config/omp.urdf (robot description, URDF)
Before this commit: robot omp, 9 links, 8 joints
Joints:
- joint joint1: limit lower=-1.57079632679 upper=1.57079632679 effort=1000 velocity=6.5 -> lower=-3.1415926 upper=3.1415926 effort=1000 velocity=6.5
- joint joint4: limit lower=-1.57079632679 upper=1.57079632679 effort=1000 velocity=6.5 -> lower=-3.1415926 upper=3.1415926 effort=1000 velocity=6.5
- joint joint6: limit lower=-1.57079632679 upper=1.57079632679 effort=1000 velocity=6.5 -> lower=-3.1415926 upper=3.1415926 effort=1000 velocity=6.5
